Commit message: Trying to tune friction params

File: xacro/caster_block.xacro (robot description, xacro)
@@ -34,5 +34,5 @@
   </link>
   <!-- pivoting axle holding the two caster axles -->
-  <joint name="pivoting_axle_joint" type="fixed">
+  <joint name="pivoting_axle_joint" type="revolute">
     <parent link="bridge_suspension"/>
     <child  link="pivoting_axle"/>
@@ -72,4 +72,5 @@
     <origin xyz="0 ${caster_track_width/2} ${caster_height_trimmer}" rpy="0 0 0"/>
     <axis xyz="0 0 1"/>
+    <dynamics damping="${axle_damping}" friction="${axle_friction}"/>
   </joint>
   <link name="A_side_caster_axle">
@@ -140,4 +141,5 @@
     <origin xyz="0 ${-caster_track_width/2} ${caster_height_trimmer}" rpy="0 0 0"/>
     <axis xyz="0 0 1"/>
+    <dynamics damping="${axle_damping}" friction="${axle_friction}"/>
   </joint>
   <link name="B_side_caster_axle">
@@ -197,8 +199,11 @@
     <mu1>1.0</mu1>
     <mu2>1.0</mu2>
-    <kp>1000000.0</kp>
-    <kd>100.0</kd>
-    <minDepth>0.001</minDepth>
-    <maxVel>1.0</maxVel>
+    <slip1>0.0</slip1>
+    <slip2>0.0</slip2>
+    <kp>10000000.0</kp>
+    <kd>100.0</kd>
+    <minDepth>0.0</minDepth>
+    <maxVel>1.0</maxVel>
+    <!--<frictionModel>cone_model</frictionModel>-->
   </gazebo>
 </robot>

File: xacro/drive_block.xacro (robot description, xacro)
@@ -93,10 +93,13 @@
   <gazebo reference="${name}_drive_wheel">
     <material>Gazebo/DarkGrey</material>
-    <mu1>2.0</mu1>
-    <mu2>2.0</mu2>
+    <mu1>1.1</mu1>
+    <mu2>1.1</mu2>
+    <slip1>0.0</slip1>
+    <slip2>0.0</slip2>
     <kp>10000000.0</kp>
     <kd>100.0</kd>
-    <minDepth>0.001</minDepth>
+    <minDepth>0.0</minDepth>
     <maxVel>1.0</maxVel>
+    <!--<frictionModel>cone_model</frictionModel>-->
   </gazebo>
 </xacro:macro>

File: xacro/properties.xacro (robot description, xacro)
@@ -7,5 +7,5 @@
   <xacro:property name="body_height"             value="0.0400"/>
   <xacro:property name="body_length"             value="0.4200"/>
-  <xacro:property name="body_mass"               value="1.0000"/> <!-- khm... -->
+  <xacro:property name="body_mass"               value="0.4000"/> <!-- khm..., was 1kg -->
   <!-- battery -->
   <xacro:property name="battery_width"           value="0.0800"/>
